File: BadgeLife/KiCad and Autorouter.kicad_sch (KiCad schematic)
At the start: 21 parts, among them SW1 Power, SW2 Dice Roll, U1 ATtiny85

Commit message: HtmlBom Generated and one footprint corrected
Parts:
- D1: footprint Diode_SMD:D_0805_2012Metric -> Diode_SMD:D_0805_2012Metric_Pad1.15x1.40mm_HandSolder
Changed lines of the file:
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@@
       (effects (font (size 1.27 1.27)) (justify right))
     )
-    (property "Footprint" "Diode_SMD:D_0805_2012Metric" (id 2) (at 139.7 45.72 90)
+    (property "Footprint" "Diode_SMD:D_0805_2012Metric_Pad1.15x1.40mm_HandSolder" (id 2) (at 139.7 45.72 90)
       (effects (font (size 1.27 1.27)) hide)
     )
@@
     )
     (path "/c2362f82-f028-401c-ab37-14d044a4d523"
-      (reference "D1") (unit 1) (value "Red") (footprint "Diode_SMD:D_0805_2012Metric")
+      (reference "D1") (unit 1) (value "Red") (footprint "Diode_SMD:D_0805_2012Metric_Pad1.15x1.40mm_HandSolder")
     )
     (path "/36fe2ac2-8e53-469f-b1bc-21fc638c4489"
